Commit message: Add attempted imu to odom scheme

File: bluerov/robots/bluerov.urdf (robot description, URDF)
Before this commit: robot bluerov, 2 links, 1 joints
Links:
- added link fcu; visual box size=0.10 .05 .01
Joints:
- added joint base_link_to_fcu: type fixed, parent base_link, child fcu, origin xyz=0 0 0 rpy=0 0 0
